Commit message: Update lynxmotion_arm.urdf

File: ros2_ws/simple_sim_movement/urdf/lynxmotion_arm.urdf (robot description, URDF)
Before this commit: robot lynxmotion_arm, 8 links, 7 joints
Joints:
- joint base_link2turret: limit (none) -> lower=-1.5 upper=1.5 effort=1000.0 velocity=3.1416; type continuous -> revolute
- joint forearm2wrist: limit (none) -> lower=-1.5 upper=1.5 effort=1000.0 velocity=3.1416; type continuous -> revolute
- joint turret2upperarm: limit (none) -> lower=-1.5 upper=1.5 effort=1000.0 velocity=3.1416; type continuous -> revolute
- joint upperarm2forearm: limit (none) -> lower=-1.5 upper=1.5 effort=1000.0 velocity=3.1416; type continuous -> revolute
- joint wrist2hand: limit (none) -> lower=-1.5 upper=1.5 effort=1000.0 velocity=3.1416; type continuous -> revolute
